Commit message: feat(description): restructure arm kinematic chain (split shoulder/elbow roll)
Split shoulder_roll into its own revolute joint via a dummy shoulder_link,
rework elbow_roll onto the forearm, make the wrist fixed, and widen leg/arm
joint limits to allow negative angles. Retune wave/bow/march poses in
pose_definitions to match the new arm chain.

Co-Authored-By: Claude Opus 4.8 <noreply@anthropic.com>

File: ros2_ws/src/my_robot_description/urdf/humanoid.urdf.xacro (robot description, xacro)
@@ -109,5 +109,5 @@
       <axis xyz="1 0 0"/>
       <!-- Limits in radians: 0° to 170° -->
-      <limit lower="0.0" upper="${170.0*pi/180}" effort="10" velocity="3.0"/>
+      <limit lower="${-170.0*pi/180}" upper="${170.0*pi/180}" effort="10" velocity="3.0"/>
       <dynamics damping="0.1" friction="0.1"/>
     </joint>
@@ -130,5 +130,5 @@
       <origin xyz="0 0 0" rpy="0 0 0"/>
       <axis xyz="0 1 0"/>
-      <limit lower="0.0" upper="${170.0*pi/180}" effort="10" velocity="3.0"/>
+      <limit lower="${-170.0*pi/180}" upper="${170.0*pi/180}" effort="10" velocity="3.0"/>
       <dynamics damping="0.1" friction="0.1"/>
     </joint>
@@ -155,5 +155,5 @@
       <origin xyz="0 0 ${-thigh_len}" rpy="0 0 0"/>
       <axis xyz="0 1 0"/>
-      <limit lower="0.0" upper="${170.0*pi/180}" effort="10" velocity="3.0"/>
+      <limit lower="${-170.0*pi/180}" upper="${170.0*pi/180}" effort="10" velocity="3.0"/>
       <dynamics damping="0.1" friction="0.1"/>
     </joint>
@@ -250,8 +250,26 @@
     <joint name="${prefix}_shoulder_pitch" type="revolute">
       <parent link="torso"/>
-      <child  link="${prefix}_upper_arm"/>
+      <child  link="${prefix}_shoulder_link"/>
       <origin xyz="0 ${reflect * (torso_width/2 + shoulder_offset_y)} ${shoulder_offset_z}" rpy="0 0 0"/>
       <axis xyz="0 1 0"/>
-      <limit lower="0.0" upper="${180.0*pi/180}" effort="5" velocity="3.0"/>
+      <limit lower="${-180.0*pi/180}" upper="${180.0*pi/180}" effort="5" velocity="3.0"/>
+      <dynamics damping="0.05" friction="0.05"/>
+    </joint>
+    <!-- Dummy link required by URDF between two co-located revolute joints.
+         Must have non-zero inertia or the physics engine will reject it. -->
+    <link name="${prefix}_shoulder_link">
+      <inertial>
+        <mass value="0.001"/>
+        <inertia ixx="1e-6" ixy="0" ixz="0" iyy="1e-6" iyz="0" izz="1e-6"/>
+      </inertial>
+    </link>
+    <!-- ── SHOULDER ROLL joint ────────────────────────── -->
+    <!-- Co-located with shoulder_pitch: origin is (0 0 0) relative to shoulder_link -->
+    <joint name="${prefix}_shoulder_roll" type="revolute">
+      <parent link="${prefix}_shoulder_link"/>
+      <child  link="${prefix}_upper_arm"/>
+      <origin xyz="0 0 0" rpy="0 0 0"/>
+      <axis xyz="1 0 0"/>
+      <limit lower="${-180.0*pi/180}" upper="${180.0*pi/180}" effort="5" velocity="3.0"/>
       <dynamics damping="0.05" friction="0.05"/>
     </joint>
@@ -269,11 +287,11 @@
       </collision>
     </link>
-    <!-- ── SHOULDER ROLL joint ────────────────────────── -->
-    <joint name="${prefix}_shoulder_roll" type="revolute">
+    <!-- ── ELBOW ROLL joint ───────────────────────────── -->
+    <joint name="${prefix}_elbow_roll" type="revolute">
       <parent link="${prefix}_upper_arm"/>
       <child  link="${prefix}_forearm"/>
       <origin xyz="0 0 ${-upper_arm_len}" rpy="0 0 0"/>
       <axis xyz="1 0 0"/>
-      <limit lower="0.0" upper="${180.0*pi/180}" effort="5" velocity="3.0"/>
+      <limit lower="${-180.0*pi/180}" upper="${180.0*pi/180}" effort="5" velocity="3.0"/>
       <dynamics damping="0.05" friction="0.05"/>
     </joint>
@@ -291,12 +309,9 @@
       </collision>
     </link>
-    <!-- ── ELBOW ROLL joint ───────────────────────────── -->
-    <joint name="${prefix}_elbow_roll" type="revolute">
+    <!-- ── WRIST (fixed) ─────────────────────────────── -->
+    <joint name="${prefix}_wrist_fixed" type="fixed">
       <parent link="${prefix}_forearm"/>
       <child  link="${prefix}_hand"/>
       <origin xyz="0 0 ${-forearm_len}" rpy="0 0 0"/>
-      <axis xyz="1 0 0"/>
-      <limit lower="0.0" upper="${180.0*pi/180}" effort="5" velocity="3.0"/>
-      <dynamics damping="0.05" friction="0.05"/>
     </joint>
     <link name="${prefix}_hand">
