Commit message: M0+M1+Phase2: verified model, base estimator, Pinocchio dynamics, torque path

File: ros2_ws/src/my_robot_description/urdf/humanoid.urdf.xacro (robot description, xacro)
@@ -73,6 +73,7 @@
        ============================================================ -->
   <!-- Inertia macro for a solid box (kg, meters) -->
-  <xacro:macro name="box_inertia" params="m x y z">
+  <xacro:macro name="box_inertia" params="m x y z ox:=0 oy:=0 oz:=0">
     <inertial>
+      <origin xyz="${ox} ${oy} ${oz}" rpy="0 0 0"/>
       <mass value="${m}"/>
       <inertia
@@ -136,5 +137,6 @@
     <link name="${prefix}_thigh">
       <xacro:box_inertia m="${thigh_mass}"
-        x="${link_thickness}" y="${link_thickness}" z="${thigh_len}"/>
+        x="${link_thickness}" y="${link_thickness}" z="${thigh_len}"
+        oz="${-thigh_len/2}"/>
       <visual>
         <!-- Offset so top of box is at joint origin (thigh hangs downward) -->
@@ -161,5 +163,6 @@
     <link name="${prefix}_shank">
       <xacro:box_inertia m="${shank_mass}"
-        x="${link_thickness}" y="${link_thickness}" z="${shank_len}"/>
+        x="${link_thickness}" y="${link_thickness}" z="${shank_len}"
+        oz="${-shank_len/2}"/>
       <visual>
         <origin xyz="0 0 ${-shank_len/2}" rpy="0 0 0"/>
@@ -220,5 +223,6 @@
     <link name="${prefix}_foot">
       <xacro:box_inertia m="${foot_mass}"
-        x="${foot_len}" y="${foot_width}" z="${foot_height}"/>
+        x="${foot_len}" y="${foot_width}" z="${foot_height}"
+        oz="${-foot_height/2}"/>
       <visual>
         <!--
@@ -276,5 +280,6 @@
     <link name="${prefix}_upper_arm">
       <xacro:box_inertia m="${upper_arm_m}"
-        x="${link_thickness}" y="${link_thickness}" z="${upper_arm_len}"/>
+        x="${link_thickness}" y="${link_thickness}" z="${upper_arm_len}"
+        oz="${-upper_arm_len/2}"/>
       <visual>
         <origin xyz="0 0 ${-upper_arm_len/2}" rpy="0 0 0"/>
@@ -298,5 +303,6 @@
     <link name="${prefix}_forearm">
       <xacro:box_inertia m="${forearm_m}"
-        x="${link_thickness}" y="${link_thickness}" z="${forearm_len}"/>
+        x="${link_thickness}" y="${link_thickness}" z="${forearm_len}"
+        oz="${-forearm_len/2}"/>
       <visual>
         <origin xyz="0 0 ${-forearm_len/2}" rpy="0 0 0"/>
@@ -444,4 +450,5 @@
     <joint name="r_hip_roll">
       <command_interface name="position"/>
+      <command_interface name="effort"/>
       <state_interface name="position">
         <param name="initial_value">0.0</param>
@@ -453,4 +460,5 @@
     <joint name="r_hip_pitch">
       <command_interface name="position"/>
+      <command_interface name="effort"/>
       <state_interface name="position">
         <param name="initial_value">0.0</param>
@@ -462,4 +470,5 @@
     <joint name="r_knee_pitch">
       <command_interface name="position"/>
+      <command_interface name="effort"/>
       <state_interface name="position">
         <param name="initial_value">0.0</param>
@@ -471,4 +480,5 @@
     <joint name="r_ankle_pitch">
       <command_interface name="position"/>
+      <command_interface name="effort"/>
       <state_interface name="position">
         <param name="initial_value">0.0</param>
@@ -480,4 +490,5 @@
     <joint name="r_ankle_roll">
       <command_interface name="position"/>
+      <command_interface name="effort"/>
       <state_interface name="position">
         <param name="initial_value">0.0</param>
@@ -490,4 +501,5 @@
     <joint name="l_hip_roll">
       <command_interface name="position"/>
+      <command_interface name="effort"/>
       <state_interface name="position">
         <param name="initial_value">0.0</param>
@@ -499,4 +511,5 @@
     <joint name="l_hip_pitch">
       <command_interface name="position"/>
+      <command_interface name="effort"/>
       <state_interface name="position">
         <param name="initial_value">0.0</param>
@@ -508,4 +521,5 @@
     <joint name="l_knee_pitch">
       <command_interface name="position"/>
+      <command_interface name="effort"/>
       <state_interface name="position">
         <param name="initial_value">0.0</param>
@@ -517,4 +531,5 @@
     <joint name="l_ankle_pitch">
       <command_interface name="position"/>
+      <command_interface name="effort"/>
       <state_interface name="position">
         <param name="initial_value">0.0</param>
@@ -526,4 +541,5 @@
     <joint name="l_ankle_roll">
       <command_interface name="position"/>
+      <command_interface name="effort"/>
       <state_interface name="position">
         <param name="initial_value">0.0</param>
@@ -536,4 +552,5 @@
     <joint name="r_shoulder_pitch">
       <command_interface name="position"/>
+      <command_interface name="effort"/>
       <state_interface name="position">
         <param name="initial_value">0.0</param>
@@ -545,4 +562,5 @@
     <joint name="r_shoulder_roll">
       <command_interface name="position"/>
+      <command_interface name="effort"/>
       <state_interface name="position">
         <param name="initial_value">0.0</param>
@@ -554,4 +572,5 @@
     <joint name="r_elbow_roll">
       <command_interface name="position"/>
+      <command_interface name="effort"/>
       <state_interface name="position">
         <param name="initial_value">0.0</param>
@@ -564,4 +583,5 @@
     <joint name="l_shoulder_pitch">
       <command_interface name="position"/>
+      <command_interface name="effort"/>
       <state_interface name="position">
         <param name="initial_value">0.0</param>
@@ -573,4 +593,5 @@
     <joint name="l_shoulder_roll">
       <command_interface name="position"/>
+      <command_interface name="effort"/>
       <state_interface name="position">
         <param name="initial_value">0.0</param>
@@ -582,4 +603,5 @@
     <joint name="l_elbow_roll">
       <command_interface name="position"/>
+      <command_interface name="effort"/>
       <state_interface name="position">
         <param name="initial_value">0.0</param>
@@ -592,4 +614,5 @@
     <joint name="head_yaw">
       <command_interface name="position"/>
+      <command_interface name="effort"/>
       <state_interface name="position">
         <param name="initial_value">0.0</param>
@@ -601,4 +624,5 @@
     <joint name="camera_pitch">
       <command_interface name="position"/>
+      <command_interface name="effort"/>
       <state_interface name="position">
         <param name="initial_value">0.0</param>
@@ -649,4 +673,5 @@
   </gazebo>
   -->
+  <!-- GROUND-TRUTH odometry of base_link (validation only, not a real sensor). -->
   <!-- IMU sensor on base_link — matches real MPU6050 location -->
   <gazebo reference="base_link">
